Commit message: WIP at radius, tried to pick up single large black piece

File: wpdchess/urdf/chesstable.urdf.xacro (robot description, xacro)
@@ -6,6 +6,6 @@
   <property name="piece_z" value="0.55" />
   <property name="pitch" value="0.05"/> <!-- 5cm pitch -->
-  <property name="piece_radius" value="0.01"/>
-  <property name="piece_length" value="0.05"/>
+  <property name="piece_radius" value="0.025"/>
+  <property name="piece_length" value="0.1"/>
   <property name="piece_mass"   value="0.005"/> <!-- MKS units => 5g -->
   <!-- row 1 location -->
@@ -22,4 +22,7 @@
   <property name="cg" value="${table_y-2.5*pitch}"/>
   <property name="ch" value="${table_y-3.5*pitch}"/>
+  <xacro:chesspiece parent="table_top_link" piecename="wch" color="Black" >
+    <origin xyz="${r1} ${ch} ${piece_z}" rpy="0 0 0" />
+  </xacro:chesspiece>
 <!--
   <xacro:chesspiece parent="table_top_link" piecename="wca" color="White" >
