Commit message: Parameterized the chess pieces, updated mass & inertia, launched full PR2

File: wpdchess/urdf/chesspiece.urdf.xacro (robot description, xacro)
@@ -9,13 +9,18 @@
     <link name="${piecename}">
       <inertial>
-	<mass value="0.01" />
+	<mass value="${piece_mass}" />
 	<!-- center of mass (com) is defined w.r.t. link local coordinate system -->
 	<origin xyz="0 0 0.025" />
-	<inertia  ixx="0.0001" ixy="0.0"  ixz="0.0"  iyy="0.0001"  iyz="0.0"  izz="0.0001" />
+	<inertia  ixx="${(3*piece_radius*piece_radius + piece_length*piece_length)*piece_mass/12}"
+		  ixy="0"
+		  ixz="0"
+		  iyy="${(3*piece_radius*piece_radius + piece_length*piece_length)*piece_mass/12}"
+		  iyz="0"
+		  izz="${piece_radius*piece_radius*piece_mass/2}"/>
       </inertial>
       <visual>
 	<origin xyz="0 0 0.025" rpy="0 0 0" />
 	<geometry>
-	  <cylinder radius="0.01" length="0.05"/>
+	  <cylinder radius="${piece_radius}" length="${piece_length}"/>
 	</geometry>
       </visual>
@@ -23,5 +28,5 @@
 	<origin xyz="0 0 0.025" rpy="0 0 0" />
 	<geometry>
-	  <cylinder radius="0.01" length="0.05"/>
+	  <cylinder radius="${piece_radius}" length="${piece_length}"/>
 	</geometry>
       </collision>

File: wpdchess/urdf/chesstable.urdf.xacro (robot description, xacro)
@@ -6,4 +6,7 @@
   <property name="piece_z" value="0.55" />
   <property name="pitch" value="0.05"/> <!-- 5cm pitch -->
+  <property name="piece_radius" value="0.01"/>
+  <property name="piece_length" value="0.05"/>
+  <property name="piece_mass"   value="0.005"/> <!-- MKS units => 5g -->
   <!-- row 1 location -->
   <property name="r1" value="${table_x-3.5*pitch}"/>

Commit message: Snapshot working IK example

File: wpdchess/urdf/chesspiece.urdf.xacro (robot description, xacro)
@@ -2,5 +2,5 @@
 <robot xmlns:xacro="http://ros.org/wiki/xacro">
   <xacro:macro name="chesspiece" params="parent piecename color *origin">
-    <joint name="${piecename}_joint}" type="floating">
+    <joint name="${piecename}_joint" type="floating">
       <insert_block name="origin" />
       <parent link="${parent}"/>
