Commit message: Created chess board

File: wpdtb/urdf/chesstable.urdf.xacro (robot description, xacro)
@@ -15,9 +15,13 @@
   <property name="leg_radius" value="0.02" />
   <property name="table_top_thickness" value="0.05"/>
-  <property name="piece_z" value="${table_z+table_height}" />
+  <property name="piece_z" value="${table_z+table_height+boardthickness}" />
   <property name="pitch" value="0.04"/> <!-- 4cm pitch -->
   <property name="piece_radius" value="0.005"/>
   <property name="piece_length" value="0.05"/>
   <property name="piece_mass"   value="0.01"/> <!-- MKS units => 10g -->
+  <property name="boardthickness" value="0.01"/>
+  <property name="square_mass"    value="1"/>
+  <property name="whitesquare_color" value="Gazebo/Rocky"/>
+  <property name="blacksquare_color" value="Gazebo/WoodFloor"/>
   <!-- row 1 location -->
   <property name="r1" value="${table_x-3.5*pitch}"/>
@@ -33,4 +37,226 @@
   <property name="cg" value="${table_y-2.5*pitch}"/>
   <property name="ch" value="${table_y-3.5*pitch}"/>
+  <xacro:macro name="square1" params="name parent color depth *origin">
+    <joint name="${name}_joint" type="fixed">
+      <insert_block name="origin" />
+      <parent link="${parent}"/>
+      <child link="${name}_link"/>
+    </joint>
+    <link name="${name}_link">
+      <inertial>
+	<mass value="${square_mass}" />
+	<inertia  ixx="${2*pitch*pitch*square_mass/12}"
+		  ixy="0"
+		  ixz="0"
+		  iyy="${2*pitch*pitch*square_mass/12}"
+		  iyz="0"
+		  izz="${2*depth*depth*square_mass/12}"/>
+      </inertial>
+      <visual>
+	<geometry>
+	  <box size="${pitch} ${pitch} ${depth}"/>
+	</geometry>
+      </visual>
+      <collision>
+	<geometry>
+	  <box size="${0.99*pitch} ${0.99*pitch} ${0.99*depth}"/>
+	</geometry>
+      </collision>
+    </link>
+    <gazebo reference="${name}_link">
+      <turnGravityOff>false</turnGravityOff>
+      <genTexCoord>true</genTexCoord>
+      <kp>100000000.0</kp>
+      <kd>1000000.0</kd>
+      <material>${color}</material>
+      <selfCollide>false</selfCollide>
+    </gazebo>
+  </xacro:macro>
+  <xacro:macro name="square4" params="name parent depth *origin">
+    <joint name="${name}_center_joint" type="fixed">
+      <insert_block name="origin" />
+      <parent link="${parent}"/>
+      <child link="${name}_center_link"/>
+    </joint>
+    <link name="${name}_center_link">
+      <inertial>
+	<mass value="${4*square_mass}" />
+	<origin xyz="0 0 ${depth/4}" rpy="0 0 0" />
+	<inertia  ixx="${2*4*pitch*pitch*4*square_mass/12}"
+		  ixy="0"
+		  ixz="0"
+		  iyy="${2*4*pitch*pitch*4*square_mass/12}"
+		  iyz="0"
+		  izz="${2*depth*depth/4*4*square_mass/12}"/>
+      </inertial>
+      <visual>
+	<origin xyz="0 0 ${depth/4}" rpy="0 0 0" />
+	<geometry>
+	  <box size="${2*pitch} ${2*pitch} ${depth/2}"/>
+	</geometry>
+      </visual>
+      <collision>
+	<origin xyz="0 0 ${depth/4}" rpy="0 0 0" />
+	<geometry>
+	  <box size="${0.99*2*pitch} ${0.99*2*pitch} ${0.99*depth/2}"/>
+	</geometry>
+      </collision>
+    </link>
+    <gazebo reference="${name}_center_link">
+      <turnGravityOff>false</turnGravityOff>
+      <genTexCoord>true</genTexCoord>
+      <kp>100000000.0</kp>
+      <kd>1000000.0</kd>
+      <material>Gazebo/Black</material>
+      <selfCollide>false</selfCollide>
+    </gazebo>
+    <xacro:square1 name="${name}_a1"
+		   parent="${name}_center_link"
+		   color="${whitesquare_color}"
+		   depth="${depth/2}">
+      <origin xyz="${-pitch/2} ${pitch/2} ${3*depth/4}" rpy="0 0 0"/>
+    </xacro:square1>
+    <xacro:square1 name="${name}_b1"
+		   parent="${name}_center_link"
+		   color="${blacksquare_color}"
+		   depth="${depth/2}">
+      <origin xyz="${-pitch/2} ${-pitch/2} ${3*depth/4}" rpy="0 0 0"/>
+    </xacro:square1>
+    <xacro:square1 name="${name}_a2"
+		   parent="${name}_center_link"
+		   color="${blacksquare_color}"
+		   depth="${depth/2}">
+      <origin xyz="${pitch/2} ${pitch/2} ${3*depth/4}" rpy="0 0 0"/>
+    </xacro:square1>
+    <xacro:square1 name="${name}_b2"
+		   parent="${name}_center_link"
+		   color="${whitesquare_color}"
+		   depth="${depth/2}">
+      <origin xyz="${pitch/2} ${-pitch/2} ${3*depth/4}" rpy="0 0 0"/>
+    </xacro:square1>
+  </xacro:macro>
+  <xacro:macro name="square16" params="name parent depth *origin">
+    <joint name="${name}_center_joint" type="fixed">
+      <insert_block name="origin" />
+      <parent link="${parent}"/>
+      <child link="${name}_center_link"/>
+    </joint>
+    <link name="${name}_center_link">
+      <inertial>
+	<mass value="${4*square_mass}" />
+	<origin xyz="0 0 ${depth/4}" rpy="0 0 0" />
+	<inertia  ixx="${2*16*pitch*pitch*4*square_mass/12}"
+		  ixy="0"
+		  ixz="0"
+		  iyy="${2*16*pitch*pitch*4*square_mass/12}"
+		  iyz="0"
+		  izz="${2*depth*depth/4*4*square_mass/12}"/>
+      </inertial>
+      <visual>
+	<origin xyz="0 0 ${depth/4}" rpy="0 0 0" />
+	<geometry>
+	  <box size="${4*pitch} ${4*pitch} ${depth/2}"/>
+	</geometry>
+      </visual>
+      <collision>
+	<origin xyz="0 0 ${depth/4}" rpy="0 0 0" />
+	<geometry>
+	  <box size="${0.99*4*pitch} ${0.99*4*pitch} ${0.99*depth/2}"/>
+	</geometry>
+      </collision>
+    </link>
+    <gazebo reference="${name}_center_link">
+      <turnGravityOff>false</turnGravityOff>
+      <genTexCoord>true</genTexCoord>
+      <kp>100000000.0</kp>
+      <kd>1000000.0</kd>
+      <material>Gazebo/Black</material>
+      <selfCollide>false</selfCollide>
+    </gazebo>
+    <xacro:square4 name="${name}_a1"
+		   parent="${name}_center_link"
+		   depth="${depth/2}">
+      <origin xyz="${-2*pitch/2} ${2*pitch/2} ${3*depth/4}" rpy="0 0 0"/>
+    </xacro:square4>
+    <xacro:square4 name="${name}_b1"
+		   parent="${name}_center_link"
+		   depth="${depth/2}">
+      <origin xyz="${-2*pitch/2} ${-2*pitch/2} ${3*depth/4}" rpy="0 0 0"/>
+    </xacro:square4>
+    <xacro:square4 name="${name}_a2"
+		   parent="${name}_center_link"
+		   depth="${depth/2}">
+      <origin xyz="${2*pitch/2} ${2*pitch/2} ${3*depth/4}" rpy="0 0 0"/>
+    </xacro:square4>
+    <xacro:square4 name="${name}_b2"
+		   parent="${name}_center_link"
+		   depth="${depth/2}">
+      <origin xyz="${2*pitch/2} ${-2*pitch/2} ${3*depth/4}" rpy="0 0 0"/>
+    </xacro:square4>
+  </xacro:macro>
+  <xacro:macro name="square64" params="name parent depth *origin">
+    <joint name="${name}_center_joint" type="fixed">
+      <insert_block name="origin" />
+      <parent link="${parent}"/>
+      <child link="${name}_center_link"/>
+    </joint>
+    <link name="${name}_center_link">
+      <inertial>
+	<mass value="${4*square_mass}" />
+	<origin xyz="0 0 ${depth/4}" rpy="0 0 0" />
+	<inertia  ixx="${2*64*pitch*pitch*4*square_mass/12}"
+		  ixy="0"
+		  ixz="0"
+		  iyy="${2*64*pitch*pitch*4*square_mass/12}"
+		  iyz="0"
+		  izz="${2*depth*depth/4*4*square_mass/12}"/>
+      </inertial>
+      <visual>
+	<origin xyz="0 0 ${depth/4}" rpy="0 0 0" />
+	<geometry>
+	  <box size="${8*pitch} ${8*pitch} ${depth/2}"/>
+	</geometry>
+      </visual>
+      <collision>
+	<origin xyz="0 0 ${depth/4}" rpy="0 0 0" />
+	<geometry>
+	  <box size="${0.99*8*pitch} ${0.99*8*pitch} ${0.99*depth/2}"/>
+	</geometry>
+      </collision>
+    </link>
+    <gazebo reference="${name}_center_link">
+      <turnGravityOff>false</turnGravityOff>
+      <genTexCoord>true</genTexCoord>
+      <kp>100000000.0</kp>
+      <kd>1000000.0</kd>
+      <material>Gazebo/Black</material>
+      <selfCollide>false</selfCollide>
+    </gazebo>
+    <xacro:square16 name="${name}_a1"
+		    parent="${name}_center_link"
+		    depth="${depth/2}">
+      <origin xyz="${-4*pitch/2} ${4*pitch/2} ${3*depth/4}" rpy="0 0 0"/>
+    </xacro:square16>
+    <xacro:square16 name="${name}_b1"
+		    parent="${name}_center_link"
+		    depth="${depth/2}">
+      <origin xyz="${-4*pitch/2} ${-4*pitch/2} ${3*depth/4}" rpy="0 0 0"/>
+    </xacro:square16>
+    <xacro:square16 name="${name}_a2"
+		    parent="${name}_center_link"
+		    depth="${depth/2}">
+      <origin xyz="${4*pitch/2} ${4*pitch/2} ${3*depth/4}" rpy="0 0 0"/>
+    </xacro:square16>
+    <xacro:square16 name="${name}_b2"
+		    parent="${name}_center_link"
+		    depth="${depth/2}">
+      <origin xyz="${4*pitch/2} ${-4*pitch/2} ${3*depth/4}" rpy="0 0 0"/>
+    </xacro:square16>
+  </xacro:macro>
+  <xacro:square64 name="gameboard"
+		  parent="table_top_link"
+		  depth="${boardthickness}">
+    <origin xyz="${table_x} ${table_y} ${table_height}" rpy="0 0 0" />
+  </xacro:square64>
 <!--
   <xacro:chesspiece parent="table_top_link" piecename="wch" color="Black" >

Commit message: Replaced 85(ish) element chessboard with a single element board.
Instead of constructing the chessboard by building a 2x2 macro,
putting 4 of those into a 4x4 macro, and putting 4 of those into an
8x8 macro, I just made a chess board out of a single box.  It doesn't
have the checkerboard pattern on it, but I think I can do that by
specifying some sort of JPG image as the "texture".

File: wpdtb/urdf/chesstable.urdf.xacro (robot description, xacro)
@@ -254,4 +254,5 @@
     </xacro:square16>
   </xacro:macro>
+<!--
   <xacro:square64 name="gameboard"
 		  parent="table_top_link"
@@ -259,4 +260,41 @@
     <origin xyz="${table_x} ${table_y} ${table_height}" rpy="0 0 0" />
   </xacro:square64>
+-->
+<joint name="board_joint" type="fixed">
+  <origin xyz="${table_x} ${table_y} ${table_height}" rpy="0 0 0" />
+  <parent link="table_top_link"/>
+  <child link="board_link"/>
+</joint>
+<link name="board_link">
+  <inertial>
+    <mass value="${64*square_mass}" />
+    <inertia ixx="${2*64*pitch*pitch*64*square_mass/12}"
+	     ixy="0"
+	     ixz="0"
+	     iyy="${2*64*pitch*pitch*64*square_mass/12}"
+	     iyz="0"
+	     izz="${2*boardthickness*boardthickness*64*square_mass/12}"/>
+  </inertial>
+  <visual>
+    <origin xyz="0 0 ${boardthickness/2}" rpy="0 0 0"/>
+    <geometry>
+      <box size="${8*pitch} ${8*pitch} ${boardthickness}" />
+    </geometry>
+  </visual>
+  <collision>
+    <origin xyz="0 0 ${boardthickness/2}" rpy="0 0 0"/>
+    <geometry>
+      <box size="${8*pitch} ${8*pitch} ${boardthickness}" />
+    </geometry>
+  </collision>
+</link>
+<gazebo reference="board_link">
+  <turnGravityOff>false</turnGravityOff>
+  <genTexCoord>true</genTexCoord>
+  <kp>100000000.0</kp>
+  <kd>1000000.0</kd>
+  <material>Gazebo/Black</material>
+  <selfCollide>false</selfCollide>
+</gazebo>
 <!--
   <xacro:chesspiece parent="table_top_link" piecename="wch" color="Black" >

Commit message: Changed the color of the box chessboard from Black to WoodPallet

File: wpdtb/urdf/chesstable.urdf.xacro (robot description, xacro)
@@ -294,5 +294,5 @@
   <kp>100000000.0</kp>
   <kd>1000000.0</kd>
-  <material>Gazebo/Black</material>
+  <material>Gazebo/WoodPallet</material>
   <selfCollide>false</selfCollide>
 </gazebo>
